File: stamp_module.sch (EAGLE design)
At the start: 14 parts

Commit message: Add files via upload
Final stamp module schematic
Parts:
- removed MICRO: PIC24FJGA010-12X12, ECE477_project:PIC24FJGA010-12X12
- added IC1: PIC24FJ128GA010-12X12, ECE477_project:PIC24FJ128GA010-12X12
- added JP1, JP2: (no value), pinhead:PINHD-2X25
- added SV1: (no value), con-lstb:MA03-1
Connections:
- new net N$10: IC1.RD10, JP1.36
- new net N$14: IC1.RA15, JP1.42
- new net N$17: IC1.TDO, JP2.4
- new net N$18: IC1.RC15, JP1.48
- new net N$19: IC1.RC12, JP1.50
- new net N$2: C1.2, SV1.2
- new net N$20: IC1.TDI, JP2.6
- new net N$21: IC1.RA3, JP2.8
- new net N$22: IC1.RA2, JP2.10
- new net N$23: IC1.RG2, JP2.12
- new net N$24: IC1.RG3, JP2.14
- new net N$25: IC1.RF6, JP2.16
- new net N$26: IC1.RF7, JP2.18
- new net N$27: IC1.RF8, JP2.20
- new net N$28: IC1.RF2, JP2.22
- new net N$29: IC1.RF3, JP2.24
- new net N$30: IC1.RF5, JP2.1
- new net N$31: IC1.RF4, JP2.3
- new net N$32: IC1.RA1, JP2.25
- new net N$33: IC1.RD14, JP2.7
- new net N$34: IC1.RB15, JP2.13
- new net N$35: IC1.RB10, JP2.33
- new net N$36: IC1.RB13, JP2.17
- new net N$37: IC1.RB12, JP2.19
- new net N$38: IC1.RF12, JP2.21
- new net N$39: IC1.RF13, JP2.23
- new net N$4: H1.5, IC1.PGC1, JP2.28
- new net N$40: IC1.RD15, JP2.5
- new net N$41: IC1.RB11, JP2.31
- new net N$42: IC1.RB14, JP2.15
- new net N$43: IC1.RB9, JP2.35
- new net N$44: IC1.RB8, JP2.37
- new net N$45: IC1.RA10, JP2.43
- new net N$46: IC1.PMA7/VREF-/RA9, JP2.45
- new net N$47: IC1.PGD2, JP2.47
- new net N$48: IC1.PGC2, JP2.49
- new net N$49: IC1.RE6, JP1.18
- new net N$5: H1.1, IC1.!MCLR, JP2.50, R2.2, S1.3, S1.4
- new net N$50: IC1.RC1, JP1.14
- new net N$51: IC1.RE5, JP1.20
- new net N$52: IC1.VDD@1, JP1.22
- new net N$53: IC1.RE7, JP1.16
- new net N$54: IC1.RC2, JP1.12
- new net N$55: IC1.RC3, JP1.10
- new net N$56: IC1.RC4, JP1.8
- new net N$57: IC1.RG6, JP1.6
- new net N$58: IC1.RG7, JP1.4
- new net N$59: IC1.RG8, JP1.2
- new net N$6: IC1.RC14, JP1.28
- new net N$60: IC1.PRG9, JP2.48
- new net N$61: IC1.RA0, JP2.42
- new net N$62: IC1.RE8, JP2.40
- new net N$63: IC1.INT2/RE9, JP2.38
- new net N$64: IC1.RB5, JP2.36
- new net N$65: IC1.RB4, JP2.34
- new net N$66: IC1.RB3, JP2.32
- new net N$67: IC1.RB2, JP2.30
- new net N$68: IC1.RE4, JP1.1
- new net N$69: IC1.RE3, JP1.3
- new net N$7: IC1.RC13, JP1.30
- new net N$70: IC1.RE2, JP1.5
- new net N$71: IC1.RG13, JP1.7
- new net N$72: IC1.RG12, JP1.9
- new net N$73: IC1.RG14, JP1.11
- new net N$74: IC1.RE1, JP1.13
- new net N$75: IC1.RE0, JP1.15
- new net N$76: IC1.RA7, JP1.17
- new net N$77: IC1.RA6, JP1.19
- new net N$78: IC1.RG0, JP1.21
- new net N$79: IC1.RG1, JP1.23
- new net N$8: IC1.RD0, JP1.32
- new net N$80: C7.1, IC1.VCAP/VDDCORE, JP1.31
- new net N$81: IC1.RF0, JP1.27
- new net N$82: IC1.RD7, JP1.33
- new net N$83: IC1.RD6, JP1.35
- new net N$84: IC1.RD5, JP1.37
- new net N$85: IC1.RD4, JP1.39
- new net N$86: IC1.RD13, JP1.41
- new net N$87: IC1.RD12, JP1.43
- new net N$88: IC1.RD3, JP1.45
- new net N$89: IC1.RD2, JP1.47
- new net N$9: IC1.RD11, JP1.34
- new net N$90: IC1.RD1, JP1.49
- new net N$91: IC1.RG15, JP1.24
- net GND: now also IC1.AVSS, IC1.VSS@1, IC1.VSS@2, IC1.VSS@3, IC1.VSS@4, IC1.VSS@5, JP1.26, JP1.46, JP2.11, JP2.29, JP2.39, JP2.46, S1.1, S1.2, SV1.1; no longer C1.2, MICRO.AVSS, MICRO.VSS@1, MICRO.VSS@2, MICRO.VSS@3, MICRO.VSS@4, MICRO.VSS@5
- net N$1: now also IC1.RF1, JP1.25; no longer C7.1, MICRO.VCAP/VDDCORE
- net N$12: now also IC1.RD9, JP1.38; no longer R2.2, S1.3, S1.4
- net N$13: now also IC1.RD8, JP1.40; no longer H1.1, MICRO.!MCLR, S1.1, S1.2
- net N$15: now also IC1.RA14, JP1.44; no longer H1.5, MICRO.PGC1
- net N$16: now also IC1.PGD1, JP2.26; no longer MICRO.PGD1
- net VDD: now also IC1.AVDD, IC1.ENVREG, IC1.VDD@2, IC1.VDD@3, IC1.VDD@4, IC1.VDD@5, JP1.29, JP2.2, JP2.27, JP2.41, JP2.44, JP2.9; no longer MICRO.AVDD, MICRO.ENVREG, MICRO.VDD@1, MICRO.VDD@2, MICRO.VDD@3, MICRO.VDD@4, MICRO.VDD@5
Other:
- moved on the sheet: C1, C2, C3, C4, C5, C6, C7, H1, LED1, R1, R2, R3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
